Commit message: 修改mybot_v3的urdf，删去因小腿减速齿轮造成的影响

File: legged_gym/resources/robots/mybot_v3/urdf/mybot_v3.urdf (robot description, URDF)
Before this commit: robot mybot_v3, 18 links, 17 joints
Joints:
- joint FL_calf_joint: limit lower=-2.69 upper=-0.91 effort=78.17 velocity=12.0 -> lower=-2.69 upper=-0.91 effort=33.5 velocity=28.0
- joint FR_calf_joint: limit lower=-2.69 upper=-0.91 effort=78.17 velocity=12.0 -> lower=-2.69 upper=-0.91 effort=33.5 velocity=28.0
- joint RL_calf_joint: limit lower=-2.69 upper=-0.91 effort=78.17 velocity=12.0 -> lower=-2.69 upper=-0.91 effort=33.5 velocity=28.0
- joint RR_calf_joint: limit lower=-2.69 upper=-0.91 effort=78.17 velocity=12.0 -> lower=-2.69 upper=-0.91 effort=33.5 velocity=28.0

Commit message: 更新urdf

File: legged_gym/resources/robots/mybot_v3/urdf/mybot_v3.urdf (robot description, URDF)
Before this commit: robot mybot_v3, 18 links, 17 joints
Links:
- link FL_calf: mass 0.23708419 -> 0.23880158
- link FR_calf: mass 0.23765586 -> 0.23880158
